Commit message: anymal_d: fix package:// paths to match repo convention
Every other URDF in example-robot-data references meshes via
  package://example-robot-data/robots/<pkg>/meshes/...
(anymal_b, anymal_c, solo, go1/2, b1, a1, talos, ur5, etc. — 65+ files).
anymal_d's URDF alone used the non-conforming form
  package://anymal_d_simple_description/meshes/...
which only resolves if a copy of anymal_d_simple_description/ happens to
sit at the exact directory package_dirs points to (the RobotLoader passes
[<share-root>/../..] as package_dirs to Pinocchio, so the self-name form
looks for the package one level above the share tree — nowhere near where
CMake actually installs it).

This commit brings the URDF in line with the rest of the repo so installs
at any CMAKE_INSTALL_PREFIX resolve meshes correctly, with no extra
symlinks or standalone copies.

Co-Authored-By: Claude Opus 4.7 (1M context) <noreply@anthropic.com>

File: robots/anymal_d_simple_description/urdf/anymal.urdf (robot description, URDF)
Before this commit: robot anymal, 96 links, 95 joints
Links:
- link LF_FOOT: geometry collision cylinder length=0.39572 radius=0.0175; collision sphere radius=0.031455
- link LF_HAA_drive: geometry visual mesh filename=package://example-robot-data/robots/anymal_d_simple_descrip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 scale=1.0 1.0 1.0
- link LF_HFE_drive: geometry collision cylinder length=0.119 radius=0.05375; visual mesh filename=package://example-robot-data/robots/anymal_d_simple_descrip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 scale=1.0 1.0 1.0
- link LF_KFE_drive: geometry collision cylinder length=0.119 radius=0.05375; visual mesh filename=package://example-robot-data/robots/anymal_d_simple_descrip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 scale=1.0 1.0 1.0
- link LF_hip_fixed: geometry visual mesh filename=package://example-robot-data/robots/anymal_d_simple_descrip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 scale=1.0 1.0 1.0
- link LF_shank_fixed: geometry collision box size=0.13283 0.08302 0.05732; collision cylinder length=0.05732 radius=0.071
- link LF_thigh_fixed: geometry collision box size=0.093 0.063 0.285; collision cylinder length=0.08313000000000001 radius=0.07
- link LH_FOOT: geometry collision cylinder length=0.39572 radius=0.0175; collision sphere radius=0.031455
- link LH_HAA_drive: geometry visual mesh filename=package://example-robot-data/robots/anymal_d_simple_descrip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 scale=1.0 1.0 1.0
- link LH_HFE_drive: geometry collision cylinder length=0.119 radius=0.05375; visual mesh filename=package://example-robot-data/robots/anymal_d_simple_descrip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 scale=1.0 1.0 1.0
- link LH_KFE_drive: geometry collision cylinder length=0.119 radius=0.05375; visual mesh filename=package://example-robot-data/robots/anymal_d_simple_descrip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 scale=1.0 1.0 1.0
- link LH_hip_fixed: geometry visual mesh filename=package://example-robot-data/robots/anymal_d_simple_descrip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 scale=1.0 1.0 1.0
- link LH_shank_fixed: geometry collision box size=0.13283 0.08302 0.05732; collision cylinder length=0.05732 radius=0.071
- link LH_thigh_fixed: geometry collision box size=0.093 0.063 0.285; collision cylinder length=0.08313000000000001 radius=0.07
- link RF_FOOT: geometry collision cylinder length=0.39572 radius=0.0175; collision sphere radius=0.031455
- link RF_HAA_drive: geometry visual mesh filename=package://example-robot-data/robots/anymal_d_simple_descrip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 scale=1.0 1.0 1.0
- link RF_HFE_drive: geometry collision cylinder length=0.119 radius=0.05375; visual mesh filename=package://example-robot-data/robots/anymal_d_simple_descrip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 scale=1.0 1.0 1.0
- link RF_KFE_drive: geometry collision cylinder length=0.119 radius=0.05375; visual mesh filename=package://example-robot-data/robots/anymal_d_simple_descrip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 scale=1.0 1.0 1.0
- link RF_hip_fixed: geometry visual mesh filename=package://example-robot-data/robots/anymal_d_simple_descrip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 scale=1.0 1.0 1.0
- link RF_shank_fixed: geometry collision box size=0.13283 0.08302 0.05732; collision cylinder length=0.05732 radius=0.071
- link RF_thigh_fixed: geometry collision box size=0.093 0.063 0.285; collision cylinder length=0.08313000000000001 radius=0.07
- link RH_FOOT: geometry collision cylinder length=0.39572 radius=0.0175; collision sphere radius=0.031455
- link RH_HAA_drive: geometry visual mesh filename=package://example-robot-data/robots/anymal_d_simple_descrip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 scale=1.0 1.0 1.0
- link RH_HFE_drive: geometry collision cylinder length=0.119 radius=0.05375; visual mesh filename=package://example-robot-data/robots/anymal_d_simple_descrip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 scale=1.0 1.0 1.0
- link RH_KFE_drive: geometry collision cylinder length=0.119 radius=0.05375; visual mesh filename=package://example-robot-data/robots/anymal_d_simple_descrip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 scale=1.0 1.0 1.0
- link RH_hip_fixed: geometry visual mesh filename=package://example-robot-data/robots/anymal_d_simple_descrip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 scale=1.0 1.0 1.0
- link RH_shank_fixed: geometry collision box size=0.13283 0.08302 0.05732; collision cylinder length=0.05732 radius=0.071
- link RH_thigh_fixed: geometry collision box size=0.093 0.063 0.285; collision cylinder length=0.08313000000000001 radius=0.07
- link base: geometry collision box size=0.894 0.1615 0.256; collision cylinder length=0.1482 radius=0.089
- link battery: geometry visual mesh filename=package://example-robot-data/robots/anymal_d_simple_descrip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 scale=1.0 1.0 1.0
- link bottom_shell: geometry visual mesh filename=package://example-robot-data/robots/anymal_d_simple_descrip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 scale=1.0 1.0 1.0
- link docking_socket: geometry visual mesh filename=package://example-robot-data/robots/anymal_d_simple_descrip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 scale=1.0 1.0 1.0
- link face_shell_front: geometry visual mesh filename=package://example-robot-data/robots/anymal_d_simple_descrip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 scale=1.0 1.0 1.0
- link face_shell_rear: geometry visual mesh filename=package://example-robot-data/robots/anymal_d_simple_descrip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 scale=1.0 1.0 1.0
- link inspection_payload_mount: geometry collision box size=0.16 0.135 0.015; visual mesh filename=package://example-robot-data/robots/anymal_d_simple_descrip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 scale=1 1 1
- link inspection_payload_pan: geometry collision box size=0.18 0.24 0.21; visual mesh filename=package://example-robot-data/robots/anymal_d_simple_descrip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 scale=1 1 1
- link inspection_payload_tilt: geometry visual mesh filename=package://example-robot-data/robots/anymal_d_simple_descrip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 scale=1 1 1
- link lidar: geometry collision cylinder length=0.1355 radius=0.07; visual mesh filename=package://example-robot-data/robots/anymal_d_simple_descrip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
- link top_shell: geometry visual mesh filename=package://example-robot-data/robots/anymal_d_simple_descrip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 scale=1.0 1.0 1.0
